File: pcb/driver-board/layouts/default/default.kicad_pcb (KiCad board)
At the start: 2 copper layers, 45 x 60 mm, 7 parts

Commit message: feat(pcb): one-shot build script; sign the board
tools/build_outputs.sh runs place -> DRC -> renders -> gerbers in a single
call, and refuses to render or ship fab output if DRC fails. --quick stops
after DRC for a fast loop.

Claude-Session: https://claude.ai/code/session_01UQXFTEy3DeBEx85CfiBq9q
Other:
- board text added: "Designed by 0x63616c"
Changed lines of the file:
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@@
+		)
+	)
+	(gr_text "Designed by 0x63616c"
+		(at 22.5 57.6 0)
+		(layer "F.SilkS")
+		(effects
+			(font
+				(size 0.9 0.9)
+				(thickness 0.135)
+			)
 		)
 	)

Commit message: fix(pcb-v1): swap male pin header for female socket
Same bug as v2: the XIAO socket rows J1/J2 were KH-2.54PH180-1X7P
(PH = Pin Header, male). The XIAO is a module with male pins soldered
in, so the board side has to be a receptacle -- FH, not PH.

  C2932700 KH-2.54PH180-1X7P-L11.5 -> C2932672 KH-2.54FH-1X7P-H8.5

In stock (2374) per the JLCPCB search API. Pad geometry is identical
between the families, so placement and routing are untouched. DRC stays
at 0 violations / 0 unconnected; fab package and all five renders
regenerated.

Also correct the stale legacy "LCSC Part" property in both boards'
layouts. atopile writes and maintains "LCSC"; "LCSC Part" is an
unmanaged leftover that still read C2932700 after the swap, so the file
contradicted itself on which part to order.

Claude-Session: https://claude.ai/code/session_01UQXFTEy3DeBEx85CfiBq9q
Parts:
- J3, J4: footprint KH_2_54_1X7_FEMALE:HDR-TH_7P-P2.54-V-M -> KH_2_54_1X7_FEMALE:HDR-TH_7P-P2.54-V-F

Commit message: chore(pcb): regenerate layouts, fab packages and renders
Both boards: 0 DRC errors, 0 warnings on v1 (four spurious silk_overlap
warnings remain on v2's C8 -- re-confirmed spurious, they are byte-identical
with the reference field moved ~24mm away), 0 unconnected pads, 0 footprint
errors, courtyard checks active and passing, and verify_fab clean.

Claude-Session: https://claude.ai/code/session_01UQXFTEy3DeBEx85CfiBq9q
Parts:
- added ?: , SPLITFLAP_MOUNT:M3_NPTH, F.Cu at (3.50, 3.50)
- added ?: , SPLITFLAP_MOUNT:M3_NPTH, F.Cu at (41.5, 3.50)
- added ?: , SPLITFLAP_MOUNT:M3_NPTH, F.Cu at (3.50, 56.5)
- added ?: , SPLITFLAP_MOUNT:M3_NPTH, F.Cu at (41.5, 56.5)
Other:
- outline, holes or cut-outs redrawn
- rule pad_to_mask_clearance: 0 -> 0.05
